File: Supplementary Files/KiCad Schematic/KiCad Schematic.kicad_sch (KiCad schematic)
At the start: 0 parts

Commit message: KiCad added voltage divider, ADC board, some microcontroller setup.
Parts:
- added C1: 1μf, symbol Device:C
- added C2: 0.1μF, symbol Device:C
- added R1: 10kOhms, symbol Device:R
- added TH1: Thermistor_NTC, symbol Device:Thermistor_NTC
- added U1: ESP32-S3-WROOM-1, RF_Module:ESP32-S3-WROOM-1, symbol RF_Module:ESP32-S3-WROOM-1
Connections:
- new net: R1.1, TH1.2
- new net: U1.1 (GND), U1.40 (GND), U1.41 (GND)
- new net +3.0V: U1.2 (3V3)
- new net +5V: C1.1, C2.1, TH1.1
- new net Earth: C1.2, C2.2, R1.2
- no-connect marks 0 -> 1
Other:
- note added: "1"
- note added: "10"
- note added: "2"
- note added: "3"
- note added: "4"
- note added: "5"
- note added: "6"
- note added: "7"
- note added: "8"
- note added: "9"
- note added: "ADC124S051"
- note added: "Bypassing capacitors to reduce noise from source. 1μF Tantalum & .1μF Ceramic Monolithic from datasheet."
- note added: "CS SCLK VA DOUT GND DIN IN4 IN1 IN3 IN2"
- note added: "IO1 recommended by datasheet for SPI"
- note added: "Jerryrigged the ADC because all online downloads required industry email signup."
- note added: "Voltage divider to find the constant resistor's share of voltage."

Commit message: KiCad added all required pin connections between ADC and Microcontroller.
Parts:
- added C3: 100nf, symbol Device:C
- added C4: 10μF, symbol Device:C
- added R2: 10kOhm, symbol Device:R
Connections:
- net +5V is gone; now on net +3.3V: C1.1, C2.1, TH1.1
- net Earth: now also U1.1 (GND), U1.40 (GND), U1.41 (GND), C3.1, C4.1
- net at U1.3 (EN): now also R2.2
- net +3.0V renamed +3.3V
- net +3.3V: now also C3.2, C4.2, R2.1
Other:
- note added: "IO pin recommended by datasheet for SPI"
- note added: "Pins correspond to correct GPIO numbers from datasheet and as specified in framework.cpp."
- note removed: "IO1 recommended by datasheet for SPI"

Commit message: Added comments and clarifications to KiCad schematic.
Other:
- note added: "Microcontroller and CAN Interface (not shown) are already installed on the CAN data node, only the connection between the thermistor circuit and ADC is shown here, not the full connection to CAN."
Changed lines of the file:
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@@
+		)
+	)
+	(text "Microcontroller and CAN Interface (not shown) \nare already installed on the CAN data node, \nonly the connection between the thermistor circuit \nand ADC is shown here, not the full connection to CAN."
+		(exclude_from_sim no)
+		(at 198.374 36.83 0)
+		(effects
+			(font
+				(size 0.635 0.635)
+			)
 		)
 	)
